File: hardware/kicad/ioboard/ioboard/relay_outputs.kicad_sch (KiCad schematic)
At the start: 0 parts

Commit message: relay-outputs: schematic capture complete, plan closed out
All 4 channels wired: K1-K4 (Panasonic ALDP105) driven by Q1-Q4 (Nexperia
MMBT3904) through R26-R33 (510ohm base / 10k pull-down pairs) and D9-D12
(1N4148 flyback), contacts broken out independently to J3 (Phoenix Contact
MC 1,5/8-ST-3,5, 8 positions). Added C21/C22 (10uF/100nF bulk+bypass) at
the 5V_RELAY entry point for EMI/noise reasons -- documented as design
decision 5, with corrected reasoning (coil inductance already rate-limits
the current step, so this isn't about regulator transient response the
way core-compute's WiFi-burst caps were).

Root sheet now wires relay_outputs' 5V_RELAY hierarchical pin to power's
output, verified programmatically that the wire path actually joins both
pin coordinates. Caught and fixed a reversed flyback diode (D9) before
commit -- would have put a forward-biased diode across the coil the whole
time each transistor was on.

Also commits the imported ALDP105 KiCad symbol/footprint library (no
numbered pinout exists in any datasheet, so pin functions were verified
live against the placed symbol, same resolution used for the LTV-247).
The imported footprint has the right pad count but has NOT been
independently checked against the real part's mechanical drawing --
flagged explicitly in the plan doc and CLAUDE.md rather than assumed
correct just because it came from a library.

Documentation: relay-outputs.md completed through sign-off (schematic
capture, verification checklist, acceptance criteria, BOM, commissioning
items), new relay_outputs_bom.csv (23 parts, CSV-parse verified), and
hardware/kicad/README.md updated. ERC and footprint assignment (including
the ALDP105 footprint check) deferred to the same pre-merge pass as
digital-inputs, per the user's standing policy -- tracked in CLAUDE.md.

Co-Authored-By: Claude Sonnet 5 <noreply@anthropic.com>
Claude-Session: https://claude.ai/code/session_011Mk4ACKLUzGL8p2SUjrweQ
Parts:
- added C21: 10uF, symbol Device:C
- added C22: 100nF, symbol Device:C
- added D10, D11, D12, D9: 1N4148, symbol Device:D
- added J3: Conn_01x08, symbol Connector_Generic:Conn_01x08
- added K1, K2, K3, K4: ALDP105, ALDP105:RELAY_ALDP105, symbol ALDP105:ALDP105
- added Q1, Q2, Q3, Q4: MMBT3904, Package_TO_SOT_SMD:SOT-23, symbol Transistor_BJT:MMBT3904
- added R26, R28, R30, R32: 510, symbol Device:R
- added R27, R29, R31, R33: 10k, symbol Device:R
Connections:
- new net: Q1.1 (B), R26.2, R27.2
- new net: D9.2 (A), K1.2, Q1.3 (C)
- new net: Q4.1 (B), R32.2, R33.2
- new net: Q3.1 (B), R30.2, R31.2
- new net: D12.2 (A), K4.2, Q4.3 (C)
- new net: Q2.1 (B), R28.2, R29.2
- new net: D10.2 (A), K2.2, Q2.3 (C)
- new net: D11.2 (A), K3.2, Q3.3 (C)
- new net: J3.1 (Pin_1), K1.3
- new net: J3.2 (Pin_2), K1.4
- new net: J3.3 (Pin_3), K2.3
- new net: J3.4 (Pin_4), K2.4
- new net: J3.5 (Pin_5), K3.3
- new net: J3.6 (Pin_6), K3.4
- new net: J3.7 (Pin_7), K4.3
- new net: J3.8 (Pin_8), K4.4
- new net 5V_RELAY: C21.1, C22.1, D10.1 (K), D11.1 (K), D12.1 (K), D9.1 (K), K1.1, K2.1, K3.1, K4.1
- new net GND_LOGIC: C21.2, C22.2, Q1.2 (E), Q2.2 (E), Q3.2 (E), Q4.2 (E), R27.1, R29.1, R31.1, R33.1
- new net RELAY1_CTRL: R26.1
- new net RELAY2_CTRL: R28.1
- new net RELAY3_CTRL: R30.1
- new net RELAY4_CTRL: R32.1
