File: hardware/kicad/ioboard/ioboard/analog_io.kicad_sch (KiCad schematic)
At the start: 14 parts, among them J4 MC 1,5/4-ST-3,5, U10 ISO1540, U11 MCP4725A0T-E/CH, U12 LM2904, U13 LM2904, U9 ADS1115IDGSR

Commit message: analog-io: ERC clean, Steps 6-9 closed, subsystem complete
KiCad ERC run on analog_io.kicad_sch (plus the directly-tied root-sheet
pin) to a fully-explained clean state: 15 findings reviewed and excluded
with a written, per-violation comment (cross-sheet power-driver false
positives, documented spare/deferred headroom, deferred GPIO assignment,
the deferred 15V_ANALOG_ISO rail) -- nothing silently suppressed.

Two real, pre-existing bugs outside this sheet were caught and fixed
along the way, both recorded in power.md's own revision history:
- Duplicate reference collision: power.kicad_sch's reverse-polarity FET
  was also Q1, colliding with relay_outputs.kicad_sch's Q1-Q4. Renamed
  to Q5 (schematic, power_bom.csv, and every prose reference in power.md
  updated to match).
- Inconsistent GND_LOGIC labeling: power.kicad_sch had one global label
  plus four stray local labels for the same net. All four converted to
  global.

Bare R_in/R_f renamed to R_in1/R_f1 by KiCad's own Annotate tool.

Steps 7 (acceptance criteria), 8 (documentation & BOM -- new
hardware/bom/analog_io_bom.csv), and 9 (sign-off) closed out. All 9
steps of this subsystem's build plan are now done.

Co-Authored-By: Claude Sonnet 5 <noreply@anthropic.com>
Claude-Session: https://claude.ai/code/session_011Mk4ACKLUzGL8p2SUjrweQ
Parts:
- renumbered R_f to R_f1, R_in to R_in1
Changed lines of the file:
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@@
 		(on_board yes)
 		(dnp no)
-		(property "Reference" "R_f"
+		(property "Reference" "R_f1"
 			(at 178.562 81.28 90)
 			(effects
@@
 			(project ""
 				(path "/a0fa9f92-ef51-408b-9617-1545f9e9dad8/ce521ae5-fae5-4047-a79f-945e6fee8e92"
-					(reference "R_f")
+					(reference "R_f1")
 					(unit 1)
 				)
@@
 		(dnp no)
 		(fields_autoplaced yes)
-		(property "Reference" "R_in"
+		(property "Reference" "R_in1"
 			(at 168.91 90.1699 0)
 			(effects
@@
 			(project ""
 				(path "/a0fa9f92-ef51-408b-9617-1545f9e9dad8/ce521ae5-fae5-4047-a79f-945e6fee8e92"
-					(reference "R_in")
+					(reference "R_in1")
 					(unit 1)
 				)
