File: hardware/kicad/ioboard/ioboard/power.kicad_sch (KiCad schematic)
At the start: 30 parts, among them J1 PWR_IN, Q1 CSD18531Q5A, U1 LM74610QDGKRQ1, U2 TVS3300DRV, U3 171013801, U4 171013801, U5 171033801

Commit message: power: further schematic refinements (C1 value, EN wiring, and other fixes)
Continued hand-editing in KiCad after the last commit -- captures the
current state of power.kicad_sch and ioboard.kicad_sch.

Co-Authored-By: Claude Sonnet 5 <noreply@anthropic.com>
Claude-Session: https://claude.ai/code/session_011Mk4ACKLUzGL8p2SUjrweQ
Parts:
- C1: value C -> 2.2uF
Changed lines of the file:
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@@
 	)
 	(junction
-		(at 195.58 120.65)
-		(diameter 0)
-		(color 0 0 0 0)
-	)
-	(junction
 		(at 185.42 120.65)
 		(diameter 0)
@@
 	)
 	(junction
-		(at 113.03 45.72)
+		(at 200.66 66.04)
 		(diameter 0)
 		(color 0 0 0 0)
 	)
 	(junction
-		(at 130.81 100.33)
+		(at 113.03 45.72)
 		(diameter 0)
 		(color 0 0 0 0)
 	)
 	(junction
-		(at 154.94 156.21)
+		(at 130.81 100.33)
 		(diameter 0)
 		(color 0 0 0 0)
 	)
 	(junction
-		(at 194.31 156.21)
+		(at 154.94 156.21)
 		(diameter 0)
 		(color 0 0 0 0)
@@
 	(wire
 		(pts
-			(xy 195.58 100.33) (xy 200.66 100.33)
+			(xy 195.58 100.33) (xy 199.39 100.33)
 		)
 		(stroke
@@
 	(wire
 		(pts
-			(xy 195.58 120.65) (xy 199.39 120.65)
-		)
-		(stroke
-			(width 0)
-			(type default)
-		)
-	)
-	(wire
-		(pts
-			(xy 241.3 66.04) (xy 256.54 66.04)
-		)
-		(stroke
-			(width 0)
-			(type default)
-		)
-	)
-	(wire
-		(pts
 			(xy 139.7 104.14) (xy 139.7 100.33)
 		)
@@
 	(wire
 		(pts
-			(xy 241.3 76.2) (xy 256.54 76.2)
-		)
-		(stroke
-			(width 0)
-			(type default)
-		)
-	)
-	(wire
-		(pts
 			(xy 153.67 138.43) (xy 153.67 135.89)
 		)
@@
 	(wire
 		(pts
-			(xy 194.31 156.21) (xy 198.12 156.21)
-		)
-		(stroke
-			(width 0)
-			(type default)
-		)
-	)
-	(wire
-		(pts
 			(xy 157.48 86.36) (xy 166.37 86.36)
 		)
@@
 	(wire
 		(pts
+			(xy 200.66 66.04) (xy 210.82 66.04)
+		)
+		(stroke
+			(width 0)
+			(type default)
+		)
+	)
+	(wire
+		(pts
+			(xy 242.57 76.2) (xy 241.3 76.2)
+		)
+		(stroke
+			(width 0)
+			(type default)
+		)
+	)
+	(wire
+		(pts
 			(xy 138.43 139.7) (xy 138.43 135.89)
 		)
@@
 	(wire
 		(pts
+			(xy 200.66 63.5) (xy 200.66 66.04)
+		)
+		(stroke
+			(width 0)
+			(type default)
+		)
+	)
+	(wire
+		(pts
 			(xy 62.23 34.29) (xy 55.88 34.29)
 		)
@@
 	(wire
 		(pts
-			(xy 196.85 66.04) (xy 210.82 66.04)
+			(xy 196.85 66.04) (xy 200.66 66.04)
 		)
 		(stroke
@@
 	(wire
 		(pts
-			(xy 194.31 135.89) (xy 199.39 135.89)
+			(xy 194.31 135.89) (xy 198.12 135.89)
 		)
 		(stroke
@@
 	(wire
 		(pts
+			(xy 242.57 66.04) (xy 241.3 66.04)
+		)
+		(stroke
+			(width 0)
+			(type default)
+		)
+	)
+	(wire
+		(pts
 			(xy 157.48 110.49) (xy 156.21 110.49)
 		)
@@
 		)
 	)
-	(label "3V3_LOGIC"
-		(at 198.12 66.04 0)
+	(label "GND_LOGIC"
+		(at 138.43 45.72 0)
 		(effects
 			(font
@@
 		)
 	)
-	(label "5V_RELAY"
-		(at 195.58 135.89 0)
+	(label "GND_LOGIC"
+		(at 173.99 120.65 0)
 		(effects
 			(font
@@
 	)
 	(label "GND_LOGIC"
-		(at 138.43 45.72 0)
+		(at 175.26 86.36 0)
 		(effects
 			(font
@@
 	)
 	(label "GND_LOGIC"
-		(at 173.99 120.65 0)
+		(at 172.72 156.21 0)
 		(effects
 			(font
@@
 		)
 	)
-	(label "GND_LOGIC"
-		(at 175.26 86.36 0)
+	(global_label "GND_LOGIC"
+		(shape input)
+		(at 38.1 41.91 0)
+		(fields_autoplaced yes)
 		(effects
 			(font
 				(size 1.27 1.27)
 			)
-			(justify left bottom)
+			(justify left)
+		)
+		(property "Intersheetrefs" "${INTERSHEET_REFS}"
+			(at 51.4267 41.91 0)
+			(effects
+				(font
+					(size 1.27 1.27)
+				)
+				(justify left)
+				(hide yes)
+			)
 		)
 	)
-	(label "GND_LOGIC"
-		(at 172.72 156.21 0)
+	(hierarchical_label "GND_ANALOG_ISO"
+		(shape output)
+		(at 242.57 76.2 0)
 		(effects
 			(font
 				(size 1.27 1.27)
 			)
-			(justify left bottom)
+			(justify left)
 		)
 	)
-	(label "GND_ANALOG_ISO"
-		(at 241.3 76.2 0)
+	(hierarchical_label "5V_RELAY"
+		(shape output)
+		(at 198.12 135.89 0)
 		(effects
 			(font
 				(size 1.27 1.27)
 			)
-			(justify left bottom)
+			(justify left)
 		)
 	)
-	(label "3V3_ANALOG_ISO"
-		(at 241.3 66.04 0)
+	(hierarchical_label "3V3_ANALOG_ISO"
+		(shape output)
+		(at 242.57 66.04 0)
 		(effects
 			(font
 				(size 1.27 1.27)
 			)
-			(justify left bottom)
+			(justify left)
 		)
 	)
-	(label "3V3_LTE"
-		(at 196.85 100.33 0)
+	(hierarchical_label "3V3_LOGIC"
+		(shape output)
+		(at 200.66 63.5 0)
 		(effects
 			(font
 				(size 1.27 1.27)
 			)
-			(justify left bottom)
+			(justify left)
 		)
 	)
-	(global_label "GND_LOGIC"
-		(shape input)
-		(at 38.1 41.91 0)
-		(fields_autoplaced yes)
+	(hierarchical_label "3V3_LTE"
+		(shape output)
+		(at 199.39 100.33 0)
 		(effects
 			(font
@@
 			(justify left)
 		)
-		(property "Intersheetrefs" "${INTERSHEET_REFS}"
-			(at 51.4267 41.91 0)
-			(effects
-				(font
-					(size 1.27 1.27)
-				)
-				(justify left)
-				(hide yes)
-			)
-		)
 	)
 	(symbol
@@
 			)
 		)
-		(property "Value" "C"
+		(property "Value" "2.2uF"
 			(at 104.394 115.316 90)
 			(effects

Commit message: core-compute: schematic capture complete, plan closed out
lteboard KiCad project created with the ESP32-S3-WROOM-1U minimum
system: power/decoupling, EN reset RC, GPIO0 boot circuit with manual
reset/boot buttons, native USB (D+/D-, CC1/CC2 termination, series
resistors), all against GND_LOGIC/3V3_LOGIC. VBUS deliberately left
unconnected -- USB stays data-only, avoiding an unarbitrated second
power path alongside the field-power rail. Module and USB connector
(Molex 216989-0001) both matched to real sourced parts. Three items
deferred to Rev-A bring-up as commissioning tests, consistent with the
power subsystem's pattern.

Also carries a small leftover fix from the power subsystem: U6's
reference designator corrected from the KiCad-assigned default (was
still showing as PS1 in the schematic file, never previously
committed).

Co-Authored-By: Claude Sonnet 5 <noreply@anthropic.com>
Claude-Session: https://claude.ai/code/session_011Mk4ACKLUzGL8p2SUjrweQ
Parts:
- renumbered PS1 to U6
Changed lines of the file:
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@@
 		(dnp no)
 		(fields_autoplaced yes)
-		(property "Reference" "PS1"
+		(property "Reference" "U6"
 			(at 226.06 58.42 0)
 			(effects
@@
 			(project ""
 				(path "/a0fa9f92-ef51-408b-9617-1545f9e9dad8/9bc843cc-645c-4034-a877-ed0cc8bfa13d"
-					(reference "PS1")
+					(reference "U6")
 					(unit 1)
 				)

Commit message: power: add isolated 15V rail (U7, RK-0515S) for analog output gain stage
Solves the 15V problem flagged during analog-io's design: U13's output gain
amplifier needed an isolated 15V supply, and 15V_ANALOG_ISO had already been
placed as a hierarchical label on its V+ pin with nothing driving it.

- Added U7 (Recom RK-0515S, isolated DC-DC, 4.5-5.5V in / 15V out / 66mA,
  3kVDC isolation) to power.kicad_sch. Verified wiring: +VIN->5V_RELAY,
  -VIN->GND_LOGIC, +VOUT->new hierarchical label 15V_ANALOG_ISO,
  -VOUT->GND_ANALOG_ISO. Confirmed -VIN and -VOUT resolve to two distinct
  nets (isolation preserved), via a from-scratch KiCad connectivity script
  (S-expression parser + coordinate-transform pin geometry + union-find net
  reconstruction) extended this session to handle single-unit symbols using
  KiCad's "_0_0" sub-symbol convention (RK-0515S), and to detect labels that
  touch a wire mid-segment rather than at an endpoint (both 5V_RELAY and
  GND_LOGIC connect to U7 this way).
- Imported the RK-0515S KiCad symbol/footprint/3D-model library
  (hardware/kicad/ioboard/libs/RK-0515S/) and registered it in
  ioboard/sym-lib-table.
- Completed the root-sheet routing in ioboard.kicad_sch: added a
  15V_ANALOG_ISO output pin to the power sheet symbol and wired it through
  to analog_io's pre-existing 15V_ANALOG_ISO input pin. This diff also
  carries the analog_io sheet symbol's own placement (pins, position) since
  the wire terminates on it and KiCad records both in the same file -
  analog_io.kicad_sch's actual circuit content is intentionally left
  untracked/excluded, as it belongs to that subsystem's own not-yet-merged
  branch.
- docs/subsystems/power.md: added the 15V-ANALOG-ISO rail and RK-0515S
  module selection entry; corrected the LM2904 load-budget row (was a single
  row on 3.3V-LOGIC with an imprecise per-amp figure - split into U12 on
  3.3V-ANALOG-ISO and U13 on 15V-ANALOG-ISO, both at the TI-datasheet-
  verified 0.7-1.2 mA dual-package draw); updated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
Parts:
- added U7: RK-0515S, RK-0515S:CONV_RK-0515S, symbol RK-0515S:RK-0515S
- renumbered Q1 to Q5
Connections:
- net 5V_RELAY: now also U7.1 (+VIN)
- net GND_ANALOG_ISO: now also U7.5 (-VOUT)
- net GND_LOGIC: now also U7.2 (-VIN)
- new net 15V_ANALOG_ISO: U7.7 (+VOUT)
