File: hardware/kicad/ioboard/ioboard/rs485.kicad_sch (KiCad schematic)
At the start: 13 parts, among them J5 Conn_01x03, U14 ACM2520-301-2P, U15 TD321S485H-A

Commit message: Add RS232 schematic capture and wire it into the root sheet
Changed lines of the file:
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@@
 	)
 	(hierarchical_label "RS485_RXD"
-		(shape input)
+		(shape output)
 		(at 30.48 35.56 180)
 		(effects
