File: hardware/kicad/ioboard/ioboard/ioboard.kicad_sch (KiCad schematic)
At the start: 0 parts

Commit message: Complete LTE subsystem: schematic capture, master-sheet integration, and the VBAT_LTE rail fix
- lte.kicad_sch: modem (EG915UEUAC-N05-SNNSA), TXB0102 UART level shifter, pre-biased
  transistor PWRKEY/RESET_N drive (Q4/Q5), SIM interface + ESD protection (D1, now with
  all 4 channels wired including the SIM VDD line), antenna matching network, VBAT
  decoupling. Two schematic-level gaps found while verifying the master-sheet integration
  (D1's unwired 4th ESD channel, two missing No-Connect flags on U4) are fixed and
  re-verified against a fresh netlist reconstruction.
- lteboard.kicad_sch: LTE sheet symbol + its 6 hierarchical pins added and checked
  pin-for-pin against lte.kicad_sch's own hierarchical labels (name + direction) - exact
  match. Not yet wired into the rest of the board; that needs roadmap steps 6 (pin
  planning) and 7 (board-to-board connector), neither started.
- Carries the VBAT_LTE rail fix from 2026-09-13 that had never been committed: renamed
  from 3V3_LTE and retapped (137k -> 115k) from ~3.3V (the exact floor of Quectel's spec,
  zero margin) to ~3.82V, matching Quectel's typical - power.md, architecture.md,
  analog-io.md, and the corresponding ioboard.kicad_sch/power.kicad_sch label+value
  changes.
- Also includes an RS485_RXD/RS485_TXD pin/direction correction on ioboard.kicad_sch's
  root sheet pins, and RS232/ioboard reference-designator re-annotation (RS232's parts
  renumbered to fit the whole-board sequence), both already sitting in the working tree.
- Docs: lte.md (full build plan through Step 7), lte_bom.csv, README.md's new LTE section,
  roadmap.md's LTE line updated from "plan drafted" to done through schematic capture/BOM.
- Removed 4 stale duplicate doc files (CLAUDE-1.md, roadmap-1.md, ethernet-1.md,
  README-1.md), confirmed byte-identical to their real counterparts before deletion.

Co-Authored-By: Claude Sonnet 5 <noreply@anthropic.com>
Other:
- sheet power ports: added VBAT_LTE; removed 3V3_LTE
Changed lines of the file:
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@@
 			)
 		)
-		(pin "RS485_RXD" input
-			(at 62.484 118.11 0)
+		(pin "RS485_TXD" input
+			(at 62.484 124.46 0)
 			(effects
 				(font
@@
 			)
 		)
-		(pin "RS485_TXD" input
-			(at 62.484 124.46 0)
+		(pin "RS485_RXD" output
+			(at 62.484 118.11 0)
 			(effects
 				(font
@@
 			)
 		)
-		(pin "3V3_LTE" output
+		(pin "VBAT_LTE" output
 			(at 64.77 43.18 0)
 			(effects
