File: hardware/kicad/ioboard/ioboard/rs232.kicad_sch (KiCad schematic)
At the start: 7 parts, among them J1 Phoenix Contact MC 1,5/3-ST-3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, U1 MAX3232EIPWR

Commit message: Complete LTE subsystem: schematic capture, master-sheet integration, and the VBAT_LTE rail fix
- lte.kicad_sch: modem (EG915UEUAC-N05-SNNSA), TXB0102 UART level shifter, pre-biased
  transistor PWRKEY/RESET_N drive (Q4/Q5), SIM interface + ESD protection (D1, now with
  all 4 channels wired including the SIM VDD line), antenna matching network, VBAT
  decoupling. Two schematic-level gaps found while verifying the master-sheet integration
  (D1's unwired 4th ESD channel, two missing No-Connect flags on U4) are fixed and
  re-verified against a fresh netlist reconstruction.
- lteboard.kicad_sch: LTE sheet symbol + its 6 hierarchical pins added and checked
  pin-for-pin against lte.kicad_sch's own hierarchical labels (name + direction) - exact
  match. Not yet wired into the rest of the board; that needs roadmap steps 6 (pin
  planning) and 7 (board-to-board connector), neither started.
- Carries the VBAT_LTE rail fix from 2026-09-13 that had never been committed: renamed
  from 3V3_LTE and retapped (137k -> 115k) from ~3.3V (the exact floor of Quectel's spec,
  zero margin) to ~3.82V, matching Quectel's typical - power.md, architecture.md,
  analog-io.md, and the corresponding ioboard.kicad_sch/power.kicad_sch label+value
  changes.
- Also includes an RS485_RXD/RS485_TXD pin/direction correction on ioboard.kicad_sch's
  root sheet pins, and RS232/ioboard reference-designator re-annotation (RS232's parts
  renumbered to fit the whole-board sequence), both already sitting in the working tree.
- Docs: lte.md (full build plan through Step 7), lte_bom.csv, README.md's new LTE section,
  roadmap.md's LTE line updated from "plan drafted" to done through schematic capture/BOM.
- Removed 4 stale duplicate doc files (CLAUDE-1.md, roadmap-1.md, ethernet-1.md,
  README-1.md), confirmed byte-identical to their real counterparts before deletion.

Co-Authored-By: Claude Sonnet 5 <noreply@anthropic.com>
Parts:
- renumbered C1 to C24, C2 to C25, C3 to C26, C4 to C27, C5 to C29, J1 to J6, U1 to U16
Changed lines of the file:
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@@
 		(dnp no)
 		(fields_autoplaced yes)
-		(property "Reference" "C5"
+		(property "Reference" "C29"
 			(at 139.7 82.5499 0)
 			(effects
@@
 		(dnp no)
 		(fields_autoplaced yes)
-		(property "Reference" "U1"
+		(property "Reference" "U16"
 			(at 99.06 52.07 0)
 			(effects
@@
 		(dnp no)
 		(fields_autoplaced yes)
-		(property "Reference" "J1"
+		(property "Reference" "J6"
 			(at 147.32 71.1199 0)
 			(effects
@@
 		(on_board yes)
 		(dnp no)
-		(property "Reference" "C1"
+		(property "Reference" "C24"
 			(at 62.484 79.502 0)
 			(effects
@@
 		(on_board yes)
 		(dnp no)
-		(property "Reference" "C2"
+		(property "Reference" "C25"
 			(at 68.834 87.376 0)
 			(effects
@@
 		(on_board yes)
 		(dnp no)
-		(property "Reference" "C3"
+		(property "Reference" "C26"
 			(at 70.358 50.292 0)
 			(effects
@@
 		(dnp no)
 		(fields_autoplaced yes)
-		(property "Reference" "C4"
+		(property "Reference" "C27"
 			(at 128.27 87.6299 0)
 			(effects
