File: hardware/kicad/lteboard/lteboard/core-compute.kicad_sch (KiCad schematic)
At the start: 0 parts

Commit message: hardware: commit the actual core-compute schematic content
The tracked file was still the bare KiCad template (8 lines, no
components) -- the real wiring only existed in KiCad's autosave
because it was never explicitly saved (Ctrl+S) before the earlier
sign-off commit. Recovered and saved in KiCad; this commits the real
3444-line sheet: U1 (ESP32-S3-WROOM-1), J1 (USB-C receptacle),
C1-C3, R1-R6, SW1-SW2, matching docs/subsystems/core-compute.md
exactly (values, references, GND_LOGIC/3V3_LOGIC nets all verified).

Co-Authored-By: Claude Sonnet 5 <noreply@anthropic.com>
Claude-Session: https://claude.ai/code/session_011Mk4ACKLUzGL8p2SUjrweQ
Parts:
- added C1: 10uF, symbol Device:C
- added C2: 0.1uF, symbol Device:C
- added C3: 1uF, symbol Device:C
- added J1: USB_C_Receptacle_USB2.0_14P, symbol Connector:USB_C_Receptacle_USB2.0_14P
- added R1, R2: 10k, symbol Device:R
- added R3, R4: 22, symbol Device:R
- added R5, R6: 5.1k, symbol Device:R
- added SW1, SW2: SW_Push, symbol Switch:SW_Push
- added U1: ESP32-S3-WROOM-1, RF_Module:ESP32-S3-WROOM-1, symbol RF_Module:ESP32-S3-WROOM-1
Connections:
- new net: R2.2, SW2.1
- new net: SW2.2, U1.27 (IO0)
- new net: R4.1, U1.21 (IO13)
- new net: J1.A7 (D-), J1.B7 (D-), R4.2
- new net: J1.B5 (CC2), R6.2
- new net: R3.1, U1.22 (IO14)
- new net: C3.2, R1.1, SW1.1, U1.3 (EN)
- new net: J1.A6 (D+), J1.B6 (D+), R3.2
- new net: J1.A5 (CC1), R5.2
- new net: J1.A4 (VBUS), J1.A9 (VBUS), J1.B4 (VBUS), J1.B9 (VBUS)
- new net 3V3_LOGIC: C1.1, C2.1, R1.2, U1.2 (3V3)
- new net GND_LOGIC: C1.2, C2.2, C3.1, J1.A1 (GND), J1.A12 (GND), J1.B1 (GND), J1.B12 (GND), J1.S1 (SHIELD), R2.1, R5.1, R6.1, SW1.2, U1.1 (GND), U1.40 (GND), U1.41 (GND)

Commit message: hardware: fix U1 footprint to the -1U (external antenna) variant
U1 was assigned RF_Module:ESP32-S3-WROOM-1 (built-in PCB antenna),
contradicting the documented decision in core-compute.md to use the
-1U module (external U.FL antenna). Corrected to
PCM_Espressif:ESP32-S3-WROOM-1U, sourced from Espressif's own KiCad
library. Value field also updated to read ESP32-S3-WROOM-1U.

Co-Authored-By: Claude Sonnet 5 <noreply@anthropic.com>
Claude-Session: https://claude.ai/code/session_011Mk4ACKLUzGL8p2SUjrweQ
Parts:
- U1: value ESP32-S3-WROOM-1 -> ESP32-S3-WROOM-1U; footprint RF_Module:ESP32-S3-WROOM-1 -> PCM_Espressif:ESP32-S3-WROOM-1U
Changed lines of the file:
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@@
 			)
 		)
-		(property "Value" "ESP32-S3-WROOM-1"
+		(property "Value" "ESP32-S3-WROOM-1U"
 			(at 126.6033 43.18 0)
 			(effects
@@
 			)
 		)
-		(property "Footprint" "RF_Module:ESP32-S3-WROOM-1"
+		(property "Footprint" "PCM_Espressif:ESP32-S3-WROOM-1U"
 			(at 124.46 68.58 0)
 			(effects

Commit message: status-indication: fix GND_LOGIC scope, add sheet + PCA9535PW component placement
- core-compute.kicad_sch: converted 5 local GND_LOGIC labels to global_label,
  matching the project convention (global labels reserved for GND_LOGIC only).
  Local scope would have left the new status-indication sheet's GND_LOGIC
  electrically isolated from the MCU's ground - a real bug caught before wiring.
- lteboard.kicad_sch / lteboard.kicad_pro: added the new status_indication
  hierarchical sheet as LTEBOARD's second child sheet.
- status_indication.kicad_sch: new sheet, components placed (PCA9535PW I2C GPIO
  expander, 6x status LED, 6x 680R LED resistor, 2x 4.7k I2C pull-up, 1x 10k INT
  pull-up, 1x 100nF decoupling cap) - not yet wired.
- Added PCA9535PW symbol/footprint/3D-model library under hardware/kicad/lteboard/libs/
  (not in KiCad's default library) and the project's sym-lib-table pointing to it,
  fixed to use ${KIPRJMOD}-relative path instead of an absolute machine path.

Deliberately not included: uncommitted analog-io changes still sitting in this
working tree (power.kicad_sch, digital_inputs.kicad_sch, relay_outputs.kicad_sch,
ioboard.kicad_pro/kicad_sch, analog_io.kicad_sch) - this branch forked before
analog-io merged, and that content already lives on the analog-io branch.
Committing it here too would duplicate it across two branches.

Co-Authored-By: Claude Sonnet 5 <noreply@anthropic.com>
Claude-Session: https://claude.ai/code/session_011Mk4ACKLUzGL8p2SUjrweQ
Changed lines of the file:
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@@
 		)
 	)
-	(label "GND_LOGIC"
-		(at 124.46 101.6 0)
+	(global_label "GND_LOGIC"
+		(shape input)
+		(at 87.63 78.74 0)
+		(fields_autoplaced yes)
 		(effects
 			(font
 				(size 1.27 1.27)
 			)
-			(justify left bottom)
+			(justify left)
+		)
+		(property "Intersheetrefs" "${INTERSHEET_REFS}"
+			(at 100.9567 78.74 0)
+			(effects
+				(font
+					(size 1.27 1.27)
+				)
+				(justify left)
+				(hide yes)
+			)
 		)
 	)
-	(label "GND_LOGIC"
-		(at 96.52 73.66 0)
+	(global_label "GND_LOGIC"
+		(shape input)
+		(at 105.41 34.29 0)
+		(fields_autoplaced yes)
 		(effects
 			(font
 				(size 1.27 1.27)
 			)
-			(justify left bottom)
+			(justify left)
+		)
+		(property "Intersheetrefs" "${INTERSHEET_REFS}"
+			(at 118.7367 34.29 0)
+			(effects
+				(font
+					(size 1.27 1.27)
+				)
+				(justify left)
+				(hide yes)
+			)
 		)
 	)
-	(label "GND_LOGIC"
-		(at 82.55 76.2 0)
+	(global_label "GND_LOGIC"
+		(shape input)
+		(at 124.46 101.6 0)
+		(fields_autoplaced yes)
 		(effects
 			(font
 				(size 1.27 1.27)
 			)
-			(justify left bottom)
+			(justify left)
+		)
+		(property "Intersheetrefs" "${INTERSHEET_REFS}"
+			(at 137.7867 101.6 0)
+			(effects
+				(font
+					(size 1.27 1.27)
+				)
+				(justify left)
+				(hide yes)
+			)
 		)
 	)
-	(label "GND_LOGIC"
-		(at 44.45 113.03 0)
+	(global_label "GND_LOGIC"
+		(shape input)
+		(at 96.52 73.66 0)
+		(fields_autoplaced yes)
 		(effects
 			(font
 				(size 1.27 1.27)
 			)
-			(justify left bottom)
+			(justify left)
+		)
+		(property "Intersheetrefs" "${INTERSHEET_REFS}"
+			(at 109.8467 73.66 0)
+			(effects
+				(font
+					(size 1.27 1.27)
+				)
+				(justify left)
+				(hide yes)
+			)
 		)
 	)
-	(label "GND_LOGIC"
-		(at 105.41 34.29 0)
+	(global_label "GND_LOGIC"
+		(shape input)
+		(at 44.45 113.03 0)
+		(fields_autoplaced yes)
 		(effects
 			(font
 				(size 1.27 1.27)
 			)
-			(justify left bottom)
+			(justify left)
+		)
+		(property "Intersheetrefs" "${INTERSHEET_REFS}"
+			(at 57.7767 113.03 0)
+			(effects
+				(font
+					(size 1.27 1.27)
+				)
+				(justify left)
+				(hide yes)
+			)
 		)
 	)

Commit message: status-indication: complete schematic capture, cross-sheet wiring, docs, and BOM
- status_indication.kicad_sch: full wiring completed (address straps, power/ground,
  I2C pull-ups, INT pull-up, decoupling, 6 LED channels). Caught and fixed two real bugs
  via full programmatic connectivity verification (every pin/net reconstructed from the
  actual file, not just visual inspection): all 6 LEDs were initially wired with reversed
  polarity (would never have lit), and a new hierarchical 3V3_LOGIC label was placed
  floating (same name, no wire, so not actually part of the net). 10 spare GPIOs marked
  with No-Connect flags.
- core-compute.kicad_sch: converted 5 local GND_LOGIC labels to global_label (same class
  of bug fixed in power.kicad_sch during analog-io's ERC pass -- would have left this new
  sheet's ground isolated from the MCU's). Added I2C_SDA/I2C_SCL (Bidirectional, on
  GPIO8/GPIO9) and 3V3_LOGIC (Passive) hierarchical labels for cross-sheet export.
  Confirmed J1's 4 VBUS pins share one schematic pin location by symbol design, so the
  existing single No-Connect flag already covers all 4 -- no gap there.
- lteboard.kicad_sch: wired the two sheet symbols together (I2C_SDA, I2C_SCL, 3V3_LOGIC),
  verified pin types match on both ends (Passive/Passive, Bidirectional/Bidirectional x2)
  and wire endpoints land exactly on the corresponding pins.
- Added docs/subsystems/status-indication.md (full build-plan writeup, Steps 1-8) and
  hardware/bom/status_indication_bom.csv (10 parts).
- docs/roadmap.md: item 5 (status indication) marked DONE; backfilled item 4 (relay
  outputs) to DONE too, since it was already complete but never marked here.
- docs/build-log.md: added the status-indication entry, and backfilled the relay-outputs
  entry that was missing.

ERC deferred to a single project-wide pass once every subsystem is built, per current
project decision (not run per-subsystem here, unlike analog-io).

Deliberately not included: uncommitted analog-io changes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
Connections:
- net I2C_SDA: now reaches U1.12 (IO8)
- net I2C_SCL: now reaches U1.17 (IO9)
- no-connect marks 0 -> 1
Changed lines of the file:
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@@
 	)
 	(junction
-		(at 44.45 110.49)
+		(at 48.26 110.49)
 		(diameter 0)
 		(color 0 0 0 0)
@@
 	)
 	(junction
+		(at 124.46 30.48)
+		(diameter 0)
+		(color 0 0 0 0)
+	)
+	(junction
 		(at 106.68 48.26)
 		(diameter 0)
@@
 		(color 0 0 0 0)
 	)
+	(no_connect
+		(at 67.31 71.12)
+	)
+	(wire
+		(pts
+			(xy 48.26 110.49) (xy 44.45 110.49)
+		)
+		(stroke
+			(width 0)
+			(type default)
+		)
+	)
 	(wire
 		(pts
@@
 	(wire
 		(pts
-			(xy 124.46 24.13) (xy 124.46 36.83)
-		)
-		(stroke
-			(width 0)
-			(type default)
-		)
-	)
-	(wire
-		(pts
-			(xy 81.28 76.2) (xy 87.63 76.2)
+			(xy 124.46 24.13) (xy 124.46 30.48)
+		)
+		(stroke
+			(width 0)
+			(type default)
+		)
+	)
+	(wire
+		(pts
+			(xy 81.28 76.2) (xy 82.55 76.2)
 		)
 		(stroke
@@
 	(wire
 		(pts
+			(xy 125.73 30.48) (xy 124.46 30.48)
+		)
+		(stroke
+			(width 0)
+			(type default)
+		)
+	)
+	(wire
+		(pts
 			(xy 106.68 86.36) (xy 109.22 86.36)
 		)
@@
 	(wire
 		(pts
-			(xy 124.46 101.6) (xy 124.46 99.06)
-		)
-		(stroke
-			(width 0)
-			(type default)
-		)
-	)
-	(wire
-		(pts
 			(xy 67.31 83.82) (xy 68.58 83.82)
 		)
@@
 	(wire
 		(pts
-			(xy 52.07 110.49) (xy 44.45 110.49)
-		)
-		(stroke
-			(width 0)
-			(type default)
-		)
-	)
-	(wire
-		(pts
-			(xy 44.45 113.03) (xy 44.45 110.49)
+			(xy 52.07 110.49) (xy 48.26 110.49)
+		)
+		(stroke
+			(width 0)
+			(type default)
+		)
+	)
+	(wire
+		(pts
+			(xy 48.26 111.76) (xy 48.26 110.49)
 		)
 		(stroke
@@
 	(wire
 		(pts
+			(xy 124.46 30.48) (xy 124.46 36.83)
+		)
+		(stroke
+			(width 0)
+			(type default)
+		)
+	)
+	(wire
+		(pts
 			(xy 99.06 40.64) (xy 99.06 34.29)
 		)
@@
 	(wire
 		(pts
-			(xy 87.63 76.2) (xy 87.63 78.74)
-		)
-		(stroke
-			(width 0)
-			(type default)
-		)
-	)
-	(wire
-		(pts
-			(xy 87.63 78.74) (xy 81.28 78.74)
+			(xy 82.55 76.2) (xy 82.55 78.74)
+		)
+		(stroke
+			(width 0)
+			(type default)
+		)
+	)
+	(wire
+		(pts
+			(xy 82.55 78.74) (xy 81.28 78.74)
 		)
 		(stroke
@@
 	(global_label "GND_LOGIC"
 		(shape input)
-		(at 87.63 78.74 0)
+		(at 82.55 78.74 0)
 		(fields_autoplaced yes)
 		(effects
@@
 		)
 		(property "Intersheetrefs" "${INTERSHEET_REFS}"
-			(at 100.9567 78.74 0)
+			(at 95.8767 78.74 0)
 			(effects
 				(font
@@
 	(global_label "GND_LOGIC"
 		(shape input)
-		(at 124.46 101.6 0)
+		(at 124.46 99.06 270)
 		(fields_autoplaced yes)
 		(effects
@@
 				(size 1.27 1.27)
 			)
-			(justify left)
+			(justify right)
 		)
 		(property "Intersheetrefs" "${INTERSHEET_REFS}"
-			(at 137.7867 101.6 0)
+			(at 124.46 112.3867 90)
 			(effects
 				(font
 					(size 1.27 1.27)
 				)
-				(justify left)
+				(justify right)
 				(hide yes)
 			)
@@
 	(global_label "GND_LOGIC"
 		(shape input)
-		(at 96.52 73.66 0)
+		(at 96.52 73.66 180)
 		(fields_autoplaced yes)
 		(effects
@@
 				(size 1.27 1.27)
 			)
-			(justify left)
+			(justify right)
 		)
 		(property "Intersheetrefs" "${INTERSHEET_REFS}"
-			(at 109.8467 73.66 0)
+			(at 83.1933 73.66 0)
 			(effects
 				(font
 					(size 1.27 1.27)
 				)
-				(justify left)
+				(justify right)
 				(hide yes)
 			)
@@
 	(global_label "GND_LOGIC"
 		(shape input)
-		(at 44.45 113.03 0)
+		(at 48.26 111.76 270)
 		(fields_autoplaced yes)
 		(effects
@@
 				(size 1.27 1.27)
 			)
-			(justify left)
+			(justify right)
 		)
 		(property "Intersheetrefs" "${INTERSHEET_REFS}"
-			(at 57.7767 113.03 0)
+			(at 48.26 125.0867 90)
 			(effects
 				(font
 					(size 1.27 1.27)
 				)
-				(justify left)
+				(justify right)
 				(hide yes)
 			)
 		)
 	)
+	(hierarchical_label "3V3_LOGIC"
+		(shape passive)
+		(at 125.73 30.48 0)
+		(effects
+			(font
+				(size 1.27 1.27)
+			)
+			(justify left)
+		)
+	)
+	(hierarchical_label "I2C_SCL"
+		(shape bidirectional)
+		(at 109.22 76.2 180)
+		(effects
+			(font
+				(size 1.27 1.27)
+			)
+			(justify right)
+		)
+	)
+	(hierarchical_label "I2C_SDA"
+		(shape bidirectional)
+		(at 109.22 73.66 180)
+		(effects
+			(font
+				(size 1.27 1.27)
+			)
+			(justify right)
+		)
+	)
