File: hardware/kicad/lteboard/lteboard/core-compute.kicad_sch (KiCad schematic)
At the start: 13 parts, among them J1 USB_C_Receptacle_USB2.0_14P, SW1 SW_Push, SW2 SW_Push, U1 ESP32-S3-WROOM-1U

Commit message: Complete WiFi subsystem: antenna path (J2 SMA jack, EARTH-bonded shield, RF pin fed by pigtail)
Parts:
- added J2: Amphenol_132163, symbol Connector:Conn_Coaxial
Connections:
- new net EARTH: J2.2 (Ext)
- no-connect marks 1 -> 2
Changed lines of the file:
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@@
 		(at 67.31 71.12)
 	)
+	(no_connect
+		(at 163.83 39.37)
+	)
 	(wire
 		(pts
@@
 		(pts
 			(xy 124.46 24.13) (xy 114.3 24.13)
+		)
+		(stroke
+			(width 0)
+			(type default)
+		)
+	)
+	(wire
+		(pts
+			(xy 168.91 48.26) (xy 168.91 44.45)
 		)
 		(stroke
@@
 				)
 				(justify right)
+				(hide yes)
+			)
+		)
+	)
+	(global_label "EARTH"
+		(shape input)
+		(at 168.91 48.26 0)
+		(fields_autoplaced yes)
+		(effects
+			(font
+				(size 1.27 1.27)
+			)
+			(justify left)
+		)
+		(property "Intersheetrefs" "${INTERSHEET_REFS}"
+			(at 177.7009 48.26 0)
+			(effects
+				(font
+					(size 1.27 1.27)
+				)
+				(justify left)
 				(hide yes)
 			)
@@
 					(unit 1)
 				)
+			)
+		)
+	)
+	(symbol
+		(lib_id "Connector:Conn_Coaxial")
+		(at 168.91 39.37 0)
+		(unit 1)
+		(exclude_from_sim no)
+		(in_bom yes)
+		(on_board yes)
+		(dnp no)
+		(fields_autoplaced yes)
+		(property "Reference" "J2"
+			(at 172.72 38.3931 0)
+			(effects
+				(font
+					(size 1.27 1.27)
+				)
+				(justify left)
+			)
+		)
+		(property "Value" "Amphenol_132163"
+			(at 172.72 40.9331 0)
+			(effects
+				(font
+					(size 1.27 1.27)
+				)
+				(justify left)
+			)
+		)
+		(property "Footprint" ""
+			(at 168.91 39.37 0)
+			(effects
+				(font
+					(size 1.27 1.27)
+				)
+				(hide yes)
+			)
+		)
+		(property "Datasheet" "~"
+			(at 168.91 39.37 0)
+			(effects
+				(font
+					(size 1.27 1.27)
+				)
+				(hide yes)
+			)
+		)
+		(property "Description" "coaxial connector (BNC, SMA, SMB, SMC, Cinch/RCA, LEMO, ...)"
+			(at 168.91 39.37 0)
+			(effects
+				(font
+					(size 1.27 1.27)
+				)
+				(hide yes)
+			)
+		)
+		(pin "1"
+		)
+		(pin "2"
+		)
+		(instances
+			(project ""
+				(path "/e3cbe890-827c-4e3e-bf4e-d33595c4d0b3/c927d60d-8176-4f24-a893-82b8dcb11c1f"
+					(reference "J2")
+					(unit 1)
+				)
