File: hardware/kicad/lteboard/lteboard/status_indication.kicad_sch (KiCad schematic)
At the start: 17 parts, among them U2 PCA9535PW

Commit message: Complete Ethernet subsystem: schematic capture done, termination network confirmed via direct datasheet read
Parts:
- renumbered D_ETH to D_ETH1, D_FLT to D_FLT1, D_HB to D_HB1, D_LTE to D_LTE1, D_PWR to D_PWR1, D_WIFI to D_WIFI1
Changed lines of the file:
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@@
 		(on_board yes)
 		(dnp no)
-		(property "Reference" "D_LTE"
+		(property "Reference" "D_LTE1"
 			(at 87.884 86.36 0)
 			(effects
@@
 			(project "lteboard"
 				(path "/e3cbe890-827c-4e3e-bf4e-d33595c4d0b3/ec8569af-218c-4aac-87d3-711148df7d45"
-					(reference "D_LTE")
+					(reference "D_LTE1")
 					(unit 1)
 				)
@@
 		(on_board yes)
 		(dnp no)
-		(property "Reference" "D_ETH"
+		(property "Reference" "D_ETH1"
 			(at 87.376 96.266 0)
 			(effects
@@
 			(project ""
 				(path "/e3cbe890-827c-4e3e-bf4e-d33595c4d0b3/ec8569af-218c-4aac-87d3-711148df7d45"
-					(reference "D_ETH")
+					(reference "D_ETH1")
 					(unit 1)
 				)
@@
 		(on_board yes)
 		(dnp no)
-		(property "Reference" "D_PWR"
+		(property "Reference" "D_PWR1"
 			(at 88.138 70.866 0)
 			(effects
@@
 			(project ""
 				(path "/e3cbe890-827c-4e3e-bf4e-d33595c4d0b3/ec8569af-218c-4aac-87d3-711148df7d45"
-					(reference "D_PWR")
+					(reference "D_PWR1")
 					(unit 1)
 				)
@@
 		(on_board yes)
 		(dnp no)
-		(property "Reference" "D_HB"
+		(property "Reference" "D_HB1"
 			(at 88.138 79.502 0)
 			(effects
@@
 			(project "lteboard"
 				(path "/e3cbe890-827c-4e3e-bf4e-d33595c4d0b3/ec8569af-218c-4aac-87d3-711148df7d45"
-					(reference "D_HB")
+					(reference "D_HB1")
 					(unit 1)
 				)
@@
 		(on_board yes)
 		(dnp no)
-		(property "Reference" "D_WIFI"
+		(property "Reference" "D_WIFI1"
 			(at 87.63 105.156 0)
 			(effects
@@
 			(project "lteboard"
 				(path "/e3cbe890-827c-4e3e-bf4e-d33595c4d0b3/ec8569af-218c-4aac-87d3-711148df7d45"
-					(reference "D_WIFI")
+					(reference "D_WIFI1")
 					(unit 1)
 				)
@@
 		(on_board yes)
 		(dnp no)
-		(property "Reference" "D_FLT"
+		(property "Reference" "D_FLT1"
 			(at 87.884 114.046 0)
 			(effects
@@
 			(project "lteboard"
 				(path "/e3cbe890-827c-4e3e-bf4e-d33595c4d0b3/ec8569af-218c-4aac-87d3-711148df7d45"
-					(reference "D_FLT")
-					(unit 1)
-				)
+					(reference "D_FLT1")
+					(unit 1)
+				)
