File: hardware/kicad/ioboard+lteboard/ioboard+lteboard/analog_io.kicad_sch (KiCad schematic)
At the start: 14 parts, among them J1 MC 1,5/4-ST-3,5, U1 LM2904, U2 ADS1115IDGSR, U3 ISO1540, U4 MCP4725A0T-E/CH, U5 LM2904

Commit message: Step 6: pin assignment and wiring on ioboard+lteboard
- core-compute: fix USB D+/D- to native GPIO19/GPIO20 (was on GPIO13/14)
- analog_io: expose ISO1540 logic-side I2C as hierarchical labels (bidirectional)
- core-compute: add 14 hierarchical labels for ethernet/lte/rs485/rs232 pin assignment
- root sheet: wire all 14 signals to their subsystems, confirm I2C 3-way merge
  (analog_io + core-compute + status_indication)
- root sheet: VBAT_LTE tied power<->lte (casual, ahead of the formal
  board-to-board connector decision, which stays a step 7 item; 3V3_LOGIC
  intentionally left split for the same reason)
Connections:
- net SCL_ISO renamed I2C_SCL
- net SDA_ISO renamed I2C_SDA
Changed lines of the file:
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@@
-		)
-	)
-	(label "SCL_ISO"
-		(at 149.86 35.56 0)
-		(effects
-			(font
-				(size 1.27 1.27)
-			)
-			(justify left bottom)
 		)
 	)
@@
 	(label "AI2"
 		(at 222.25 77.47 0)
-		(effects
-			(font
-				(size 1.27 1.27)
-			)
-			(justify left bottom)
-		)
-	)
-	(label "SDA_ISO"
-		(at 149.86 33.02 0)
 		(effects
 			(font
@@
 		)
 	)
+	(hierarchical_label "I2C_SCL"
+		(shape bidirectional)
+		(at 149.86 35.56 0)
+		(effects
+			(font
+				(size 1.27 1.27)
+			)
+			(justify left)
+		)
+	)
 	(hierarchical_label "GND_ANALOG_ISO"
 		(shape input)
@@
 		)
 	)
+	(hierarchical_label "I2C_SDA"
+		(shape bidirectional)
+		(at 149.86 33.02 0)
+		(effects
+			(font
+				(size 1.27 1.27)
+			)
+			(justify left)
+		)
+	)

Commit message: Close roadmap steps 6/7: pin assignment, board-to-board wiring, ERC pass clean; update docs to match
Connections:
- no-connect marks 0 -> 3
Changed lines of the file:
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@@
 		(color 0 0 0 0)
+	)
+	(no_connect
+		(at 106.68 69.85)
+	)
+	(no_connect
+		(at 86.36 77.47)
+	)
+	(no_connect
+		(at 86.36 80.01)
 	)
 	(wire
