File: hardware/kicad/ioboard+lteboard/ioboard+lteboard/lte.kicad_sch (KiCad schematic)
At the start: 37 parts, among them J3 Conn_Coaxial, J4 SF53S006VCBR2000, Q4 Q_NPN, Q5 Q_NPN, U4 EG915UEUAC-N05-SNNSA, U5 TXB0102DCUR

Commit message: Merge ioboard and lteboard into one schematic project named ioboard+lteboard
Parts:
- removed C11, C13, C19, C22: 100nF, symbol Device:C
- removed C16, C17, C18, C20, C23: 33pF, symbol Device:C
- removed C21, C24: 10pF, symbol Device:C
- removed C26: 10nF, symbol Device:C
- removed D1: ESDA6V1BC6, ESDA6V1BC6:SOT95P280X145-6N, symbol ESDA6V1BC6:ESDA6V1BC6
- removed D3: SMAJ5.0A, Diode_SMD:D_SMA, symbol Diode:SMAJ5.0A
- removed D4: D_TVS, symbol Device:D_TVS
- removed J3: Conn_Coaxial, symbol Connector:Conn_Coaxial
- removed J4: SF53S006VCBR2000, CONN_SF53S006VCBR2000_JAE, symbol SF53S006VCBR2000:SF53S006VCBR2000
- removed Q4, Q5: Q_NPN, symbol Device:Q_NPN
- removed R22: 10k, symbol Device:R
- removed R25, R29, R30, R32: 0, symbol Device:R
- removed R28: 15k, symbol Device:R
- removed R31: 120k, symbol Device:R
- removed R33, R35: 4.7k, symbol Device:R
- removed R34, R36: 47k, symbol Device:R
- removed U4: EG915UEUAC-N05-SNNSA, EG915UEUAC-N05-SNNSA:XCVR_EG915UEUAC-N05-SNNSA, symbol EG915U-EU:EG915UEUAC-N05-SNNSA
- removed U5: TXB0102DCUR, DCU0008A_N, symbol TI TXB0102DCUR:TXB0102DCUR
- added C36: 10nF, symbol Device:C
- added C37, C39, C41, C42, C46: 33pF, symbol Device:C
- added C38, C43, C44, C45: 100nF, symbol Device:C
- added C40, C47: 10pF, symbol Device:C
- added D18: D_TVS, symbol Device:D_TVS
- added D19: SMAJ5.0A, Diode_SMD:D_SMA, symbol Diode:SMAJ5.0A
- added D20: ESDA6V1BC6, ESDA6V1BC6:SOT95P280X145-6N, symbol ESDA6V1BC6:ESDA6V1BC6
- added J10: SF53S006VCBR2000, CONN_SF53S006VCBR2000_JAE, symbol SF53S006VCBR2000:SF53S006VCBR2000
- added J9: Conn_Coaxial, symbol Connector:Conn_Coaxial
- added Q6, Q7: Q_NPN, symbol Device:Q_NPN
- added R49, R50: 4.7k, symbol Device:R
- added R51, R52: 47k, symbol Device:R
- added R53, R54, R55, R56: 0, symbol Device:R
- added R57: 15k, symbol Device:R
- added R58: 120k, symbol Device:R
- added R59: 10k, symbol Device:R
- added U19: EG915UEUAC-N05-SNNSA, EG915UEUAC-N05-SNNSA:XCVR_EG915UEUAC-N05-SNNSA, symbol EG915U-EU:EG915UEUAC-N05-SNNSA
- added U20: TXB0102DCUR, DCU0008A_N, symbol TI TXB0102DCUR:TXB0102DCUR
- renumbered C0603 to C35, CO604 to CO1
Connections:
- net 3V3_LOGIC: now also C44.2, U20.7 (VCCB)
- net ANT_MAIN: now also R53.1, U19.60 (ANT_MAIN)
- net EARTH: now also D18.1 (A1), J9.2 (Ext)
- net GND: now also C36.2, C37.1, C38.2, C39.2, C40.2, C41.2, C42.1, C43.2, C44.1, C45.2, C46.2, C47.2, D19.2 (A2), D20.2, D20.5, J10.C5, Q6.E, Q7.E, R51.2, R52.2, R58.2, U19.100 (GND), U19.101 (GND), U19.102 (GND), U19.3 (GND), U19.31 (GND), U19.47 (USIM1_GND), U19.48 (GND), U19.50 (GND), U19.54 (GND), U19.55 (GND), U19.58 (GND), U19.59 (GND), U19.61 (GND), U19.62 (GND), U19.67 (GND), U19.68 (GND), U19.69 (GND), U19.70 (GND), U19.71 (GND), U19.72 (GND), U19.73 (GND), U19.74 (GND), U19.79 (GND), U19.80 (GND), U19.81 (GND), U19.82 (GND), U19.89 (GND), U19.90 (GND), U19.91 (GND), U20.2 (GND)
- net LTE_PWRKEY: now also R50.1
- net LTE_RESET: now also R49.1
- net LTE_RXD: now also U20.8 (B1)
- net LTE_TXD: now also U20.1 (B2)
- net MAIN_RXD: now also U19.34 (MAIN_RXD), U20.4 (A2)
- net MAIN_TXD: now also U19.35 (MAIN_TXD), U20.5 (A1)
- net USIM1_CLK: now also C37.2, D20.6, J10.C3, R55.2
- net USIM1_DATA: now also C42.2, D20.1, J10.C7, R56.2, R57.2
- net USIM1_RST: now also C41.1, D20.3, J10.C2, R54.2
- net USIM1_VDD: now also C43.1, D20.4, J10.C1, R57.1, U19.43 (USIM1_VDD)
- net VBAT_BB: now also C38.1, C39.1, C40.1, C45.1, C46.1, C47.1, D19.1 (A1), U19.32 (VBAT_BB), U19.33 (VBAT_BB), U19.52 (VBAT_RF), U19.53 (VBAT_RF)
- net VDD_EXT: now also R59.1, U19.29 (VDD_EXT), U20.3 (VCCA)
- net at CO1.1: now also D18.2 (A2), J9.1 (In), R53.2
- new net: R58.1, R59.2, U20.6 (OE)
- new net: R55.1, U19.46 (USIM1_CLK)
- new net: Q6.B, R49.2, R51.1
- new net: R54.1, U19.44 (USIM1_RST)
- new net: Q6.C, U19.17 (~{RESET})
- new net: Q7.B, R50.2, R52.1
- new net: C36.1, Q7.C, U19.15 (PWRKEY)
- new net: R56.1, U19.45 (USIM1_DATA)
- new net: U19.103 (RESERVED), U19.104 (RESERVED), U19.105 (RESERVED), U19.106 (RESERVED), U19.107 (RESERVED), U19.108 (RESERVED), U19.109 (RESERVED), U19.11 (RESERVED), U19.110 (RESERVED), U19.111 (RESERVED), U19.112 (RESERVED), U19.113 (RESERVED), U19.114 (RESERVED), U19.115 (RESERVED), U19.116 (RESERVED), U19.117 (RESERVED), U19.118 (RESERVED), U19.12 (RESERVED), U19.123 (RESERVED), U19.124 (RESERVED), U19.125 (RESERVED), U19.13 (RESERVED), U19.14 (RESERVED), U19.16 (RESERVED), U19.49 (RESERVED), U19.51 (RESERVED), U19.57 (RESERVED), U19.63 (RESERVED), U19.65 (RESERVED), U19.66 (RESERVED), U19.78 (RESERVED), U19.92 (RESERVED), U19.93 (RESERVED), U19.94 (RESERVED), U19.95 (RESERVED), U19.97 (RESERVED), U19.98 (RESERVED), U19.99 (RESERVED)
Other:
- moved on the sheet: C35, CO1, C_BYPASS1, C_bulk3, C_bulk4

Commit message: Close roadmap steps 6/7: pin assignment, board-to-board wiring, ERC pass clean; update docs to match
Connections:
- no-connect marks 45 -> 46
Changed lines of the file:
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@@
+	)
+	(no_connect
+		(at 74.93 121.92)
 	)
 	(no_connect
